File: hardware/stm32-shift-display.kicad_sch (KiCad schematic)
At the start: 43 parts, among them J1 HDR_SWD, J2 USB_C_Receptacle_USB2.0_16P, SW1 SW_PUSH, SW2 SW_PUSH, SW3 SW_PUSH, SW4 SW_PUSH, SW5 218-2LPSTR, U1 AMS1117-3.3, U2 STM32F103C8T6, X1 OT32258MJBA4SL, X2 OK322532.768KJBA4SL

Commit message: update readme
Other:
- note added: "Battery Backup for RTC & X2"
- note added: "Mounting Holes"
- note added: "STM32F103C8 Shifting Character Display"
- note added: "USB Power Regulation"
- note added: "User LEDs"
- moved on the sheet: C18, C3, C4, C5, D1, D2, D3, D4, H1, H2, H3, H4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

Commit message: Pre-autoroute on rev2
Parts:
- removed C18: SCMR22C155PRBA0, Mouser:SCMR22C155PRBA0, symbol Device:C_Polarized
- removed C2: 100n, Capacitor_SMD:C_0402_1005Metric, symbol Device:C_Small
- removed D4: BAT43, Diode_THT:D_DO-35_SOD27_P7.62mm_Horizontal, symbol Diode:BAT43
- removed H1, H2, H3, H4: M3, MountingHole:MountingHole_3.2mm_M3_Pad_Via, symbol Mechanical:MountingHole_Pad
- removed J2: USB_C_Receptacle_USB2.0_16P, Connector_USB:USB_C_Receptacle_HCTL_HC-TYPE-C-16P-01A, symbol Connector:USB_C_Receptacle_USB2.0_16P
- removed JP1: SolderJumper_2_Open, Jumper:SolderJumper-2_P1.3mm_Open_RoundedPad1.0x1.5mm, symbol Jumper:SolderJumper_2_Open
- removed R4, R5: 220R, Resistor_SMD:R_0603_1608Metric, symbol Device:R
- removed R61: 22R, Resistor_THT:R_Axial_DIN0207_L6.3mm_D2.5mm_P7.62mm_Horizontal, symbol Device:R
- removed X2: OK322532.768KJBA4SL, Crystal:Crystal_SMD_3225-4Pin_3.2x2.5mm, symbol Oscillator:ASCO
- added BT1: 1060TR, Battery:BatteryHolder_Keystone_1060_1x2032, symbol Device:Battery_Cell
- added C10, C9: 6p, Capacitor_SMD:C_0402_1005Metric, symbol Device:C_Small
- added C8: 100n, Capacitor_SMD:C_0402_1005Metric, symbol Device:C_Small
- added H1, H2, H3, H4: M3, MountingHole:MountingHole_3.2mm_M3_ISO7380, symbol Mechanical:MountingHole
- added J1: GT-USB-7010ASV, easyeda2kicad:USB-C-SMD_G-SWITCH_GT-USB-7010ASV, symbol easyeda2kicad:GT-USB-7010ASV
- added J3: HDR_UART, Connector_PinHeader_2.54mm:PinHeader_1x05_P2.54mm_Vertical, symbol Connector_Generic:Conn_01x05
- added RN13: 220R, Resistor_SMD:R_Array_Convex_4x0603, symbol Device:R_Pack04
- added U1: USBLC6-2P6, Package_TO_SOT_SMD:SOT-666, symbol Power_Protection:USBLC6-2P6
- added Y1: Q13FC13500002, Crystal:Crystal_SMD_3215-2Pin_3.2x1.5mm, symbol Device:Crystal
- C1: renamed from C7; JLCPCB Part C307331 -> (none); LCSC Part (none) -> C307331; MFR Part CL05B104KB54PNC -> (none)
- C11: renamed from C3; JLCPCB Part C28233 -> (none); LCSC Part (none) -> C28233
- C12: renamed from C4; JLCPCB Part C28233 -> (none); LCSC Part (none) -> C28233
- C13: renamed from C5; JLCPCB Part C7171 -> (none); LCSC Part (none) -> C7171; MFR Part TAJA106K016RNJ -> (none)
- C2: renamed from C8; JLCPCB Part C307331 -> (none); LCSC Part (none) -> C307331; MFR Part CL05B104KB54PNC -> (none)
- C3: renamed from C9; JLCPCB Part C307331 -> (none); LCSC Part (none) -> C307331; MFR Part CL05B104KB54PNC -> (none)
- C4: renamed from C10; JLCPCB Part C307331 -> (none); LCSC Part (none) -> C307331; MFR Part CL05B104KB54PNC -> (none)
- C5: renamed from C11; JLCPCB Part C307331 -> (none); LCSC Part (none) -> C307331; MFR Part CL05B104KB54PNC -> (none)
- C6: JLCPCB Part C307331 -> (none); LCSC Part (none) -> C307331; MFR Part CL05B104KB54PNC -> (none)
- C7: renamed from C1; JLCPCB Part C307331 -> (none); LCSC Part (none) -> C307331; MFR Part CL05B104KB54PNC -> (none)
- D1, D2, D3: value KT-0805Y -> LED_YLW; footprint LED_SMD:LED_0805_2012Metric -> LED_THT:LED_D3.0mm; JLCPCB Part C2296 -> (none)
- R1: JLCPCB Part C25744 -> (none); LCSC Part (none) -> C25744
- R2: renamed from R7; JLCPCB Part C25905 -> (none); LCSC Part (none) -> C25905
- R3: renamed from R8; JLCPCB Part C25905 -> (none); LCSC Part (none) -> C25905
- R4: renamed from R9; value 10R -> 0R; JLCPCB Part C25077 -> (none); LCSC Part (none) -> C17168
- R5: renamed from R10; value 10R -> 0R; JLCPCB Part C25077 -> (none); LCSC Part (none) -> C17168
- R6: value 220R -> 1k5; footprint Resistor_SMD:R_0603_1608Metric -> Resistor_SMD:R_0402_1005Metric; JLCPCB Part C22962 -> (none); LCSC Part (none) -> C25867; MFR Part 0603WAF2200T5E -> (none)
- R7: renamed from R2; JLCPCB Part C25744 -> (none); LCSC Part (none) -> C25744
- R8: renamed from R3; JLCPCB Part C25744 -> (none); LCSC Part (none) -> C25744
- SW1: renamed from SW4; value SW_PUSH -> TS-1101-C-W; footprint Button_Switch_THT:SW_PUSH_6mm -> easyeda2kicad:SW-SMD_L6.0-W3.3-LS8.0; LCSC Part (none) -> C318938
- SW2: renamed from SW1; footprint Button_Switch_THT:SW_PUSH_6mm -> Mouser:TS046643BK160SMT; MFR Part (none) -> TS04-66-73-BK-260-SMT; Mouser Part (none) -> 179-TS046673BK260SMT
- SW3: renamed from SW2; footprint Button_Switch_THT:SW_PUSH_6mm -> Mouser:TS046643BK160SMT; MFR Part (none) -> TS04-66-73-BK-260-SMT; Mouser Part (none) -> 179-TS046673BK260SMT
- SW4: renamed from SW3; footprint Button_Switch_THT:SW_PUSH_6mm -> Mouser:TS046643BK160SMT; MFR Part (none) -> TS04-66-73-BK-260-SMT; Mouser Part (none) -> 179-TS046673BK260SMT
- SW5: JLCPCB Part C2961921 -> (none); LCSC Part (none) -> C2961921
- U2: JLCPCB Part C8734 -> (none); LCSC Part (none) -> C8734
- U3: renamed from U1; JLCPCB Part C6186 -> (none); LCSC Part (none) -> C6186
- X1: JLCPCB Part C717687 -> (none); LCSC Part (none) -> C717687
- renumbered J1 to J2
Connections:
- net BTN1: now also U2.39 (PB3); no longer U2.13 (PA3)
- net BTN2: now also U2.40 (PB4); no longer U2.14 (PA4)
- net BTN3: now also U2.41 (PB5); no longer U2.15 (PA5)
- net CC1: now also J1.A5 (CC1)
- net CC2: now also J1.B5 (CC2)
- net GND: now also BT1.2 (-), C10.1, C8.2, C9.1, J1.1 (SHELL), J1.2 (SHELL), J1.3 (SHELL), J1.4 (SHELL), J1.A1B12 (GND), J1.B1A12 (GND), J3.5 (Pin_5), U1.2 (GND)
- net LED1: now also U2.42 (PB6), RN13.4 (R4.1); no longer U2.12 (PA2)
- net LED1r: now also RN13.5 (R4.2)
- net LED2: now also U2.43 (PB7), RN13.3 (R3.1); no longer U2.11 (PA1)
- net LED2r: now also RN13.6 (R3.2)
- net LED3: now also U2.45 (PB8), RN13.2 (R2.1); no longer R6.2, U2.10 (PA0)
- net LED3r: now also RN13.7 (R2.2); no longer R6.1
- net OSC32_IN: now also C9.2, Y1.2
- net Shift Display/RCLK: now also U2.12 (PA2); no longer U2.42 (PB6)
- net Shift Display/SER: now also U2.13 (PA3); no longer U2.39 (PB3)
- net Shift Display/SRCLK: now also U2.14 (PA4); no longer U2.40 (PB4)
- net Shift Display/~{OE}: now also U2.10 (PA0); no longer U2.43 (PB7)
- net Shift Display/~{SRCLR}: now also U2.11 (PA1); no longer U2.41 (PB5)
- net USB_D+: now also J1.A6 (DP1), J1.B6 (DP2), U1.3 (I/O2); no longer R5.2
- net USB_D-: now also J1.A7 (DN1), J1.B7 (DN2), U1.1 (I/O1); no longer R4.2
- net VBAT: now also BT1.1 (+)
- net VBUS: now also C8.1, J1.A4B9 (VBUS), J1.B4A9 (VBUS), U1.5 (VBUS)
- net VCC: now also R6.1
- net TX3: now reaches U2.21 (PB10)
- net TX3: now also J3.1 (Pin_1)
- net RX3: now reaches U2.22 (PB11)
- net RX3: now also J3.2 (Pin_2)
- net CTS3: now reaches U2.26 (PB13)
- net CTS3: now also J3.3 (Pin_3)
- net RTS3: now reaches U2.27 (PB14)
- net RTS3: now also J3.4 (Pin_4)
- net OSC32_OUT: now reaches U2.4 (PC15)
- net OSC32_OUT: now also C10.2, Y1.1
- new net ESD_D+: R5.2, R6.2, U1.4 (I/O2)
- new net ESD_D-: R4.2, U1.6 (I/O1)
- no-connect marks 24 -> 19
Other:
- note added: "Battery Backup for RTC"
- note added: "User Buttons"
- note removed: "Battery Backup for RTC & X2"
- moved on the sheet: C11, C12, C13, D1, D2, D3, R2, R3, R4, R5, R7, R8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

Commit message: Initial rev2 design, layout, routing, and mech done. Order submitted.
Parts:
- removed RN13: 220R, Resistor_SMD:R_Array_Convex_4x0603, symbol Device:R_Pack04
- added R59, R60, R61: 220R, Resistor_SMD:R_0603_1608Metric, symbol Device:R_Small
Connections:
- net LED1: now also R59.2
- net LED1r: now also R59.1
- net LED2: now also R60.2
- net LED2r: now also R60.1
- net LED3: now also R61.2
- net LED3r: now also R61.1
- no-connect marks 19 -> 17
Other:
- note added: "Sponsored By"
- moved on the sheet: BT1, C11, C12, C13, H1, H2, H3, H4, U3
